Commit message: first commit

File: eva_mars_description/urdf/eva_mars.urdf (robot description, URDF)
Before this commit: robot eva_mars, 16 links, 15 joints
Links:
- added link camera_linkdrill; collision box size=0.015 0.031 0.027; visual mesh filename=package://eva_mars_description/meshes/camera.stl scale=0.0011 0.0011 0.0011
- added link camera_rgb_optic_framelo
Joints:
- added joint camera_box_joint: type fixed, parent sondaj_box_link, child camera_linkdrill, origin xyz=0.032 0.0 0.022 rpy=0 1.57 0
- added joint camera_rgb_optic_jointlo: type fixed, parent camera_linkdrill, child camera_rgb_optic_framelo, origin xyz=0 0 0 rpy=0 0 0
- joint sondaj2_joint: limit lower=-0.10 upper=0.00 effort=10.0 velocity=0.5 -> lower=-0.10 upper=0.00 effort=10.0 velocity=0.3
- joint sondaj3_joint: limit lower=-0.24 upper=0.00 effort=10.0 velocity=0.5 -> lower=-0.24 upper=0.00 effort=10.0 velocity=0.3
- joint sondaj_joint: limit lower=-0.04 upper=0.01 effort=10.0 velocity=0.5 -> lower=-0.04 upper=0.01 effort=10.0 velocity=0.3
